File: elrs_ss25_hajibarakat.kicad_sch (KiCad schematic)
At the start: 1 part, among them U1 ESP32-PICO-D4

Commit message: Add files via upload
Parts:
- added C10, C11, C5, C6: 100nF, symbol Device:C
- added C2, C3, C7, C8: 10nF, symbol Device:C
- added C4, C9: 470nF, symbol Device:C
- added L1, L2: 15uH, symbol Device:L
- added U2, U3: ~, symbol New_Library:SX1281
- added Y1, Y2: Crystal_GND24, symbol Device:Crystal_GND24
Connections:
- net +3.3V: now reaches U1.1 (VDDA), U1.43 (VDDA), U1.46 (VDDA)
- net +3.3V: now also U1.19 (VDD3P3_RTC), U1.3 (VDDA3P3), U1.37 (VDD3P3_CPU), U1.4 (VDDA3P3), U1.9 (EN), C10.1, C11.1, C3.2, C4.1, C5.1, C6.1, C7.2, C9.1, L1.2, L2.2, U2.11 (VBAT_IO), U2.12 (DCC_FB), U2.15 (VBAT), U2.2 (VDD_IN), U3.11 (VBAT_IO), U3.12 (DCC_FB), U3.15 (VBAT), U3.2 (VDD_IN)
- net CS0: now reaches U1.22 (IO2)
- net CS1: now reaches U1.34 (IO5)
- net SCK: now reaches U1.35 (IO18)
- net SCK: now also U2.18 (SCK_RTSN), U3.18 (SCK_RTSN)
- net MOSI: now reaches U1.36 (IO23)
- net MOSI: now also U2.17 (MOSI_RX), U3.17 (MOSI_RX)
- net MISO: now reaches U1.38 (IO19)
- net MISO: now also U2.16 (MISO_TX), U3.16 (MISO_TX)
- net GND: now reaches U1.49 (GND)
- net GND: now also C10.2, C11.2, C2.1, C3.1, C4.2, C5.2, C6.2, C7.1, C8.1, C9.2, U2.13 (GND), U2.20 (GND), U2.21 (GND), U2.23 (GND), U2.24 (GND), U2.5 (GND), U3.13 (GND), U3.20 (GND), U3.21 (GND), U3.23 (GND), U3.24 (GND), U3.5 (GND), Y1.2, Y1.4, Y2.2, Y2.4
- new net: L1.1, U2.14 (DCC_SW)
- new net: C8.2, U3.1 (VR_PA)
- new net: L2.1, U3.14 (DCC_SW)
- new net: U3.4 (XTA), Y2.3
- new net: U3.6 (XTB), Y2.1
- new net: U2.6 (XTB), Y1.1
- new net: U2.4 (XTA), Y1.3
- new net: C2.2, U2.1 (VR_PA)
- new net CSO: U2.19 (NSS_CTS), U3.19 (NSS_CTS)
- new net NRESET: U2.3 (NRESET), U3.3 (NRESET)
- no-connect marks 0 -> 14
Other:
- moved on the sheet: U1
